File: kicad/halo.kicad_pcb (KiCad board)
At the start: 2 copper layers, 253.7 x 96.8 mm, 92 parts, among them J1 USB_header, J2 USB_C_Receptacle_USB2.0, J3 12V_DC, P1 LED, P2 FTDI, P3 SPI, P4 LED_OUT, SW1 RST, SW2 MODE, U1 ATMEGA328, U2 LM1117-5.0, X1 16MHz

Commit message: added kicad PCB wip
Parts:
- moved C9 54.4 mm to (22.0, -34.4), turned to 90 degrees
- moved P2 54.4 mm to (26.9, -29.1)
- moved R1 50.4 mm to (34.9, -34.4), turned to 90 degrees
- moved R4 49.4 mm to (49.8, -8.76), turned to 90 degrees
- moved SW1 48.9 mm to (34.8, -25.9)
- moved C2 48.8 mm to (56.3, -27.1)
- moved B19 48.5 mm to (60.6, -24.5)
- moved D34 47.8 mm to (58.4, -27.1)
- moved R8 47.8 mm to (60.6, -27.1)
- moved B18 47.2 mm to (60.8, -22.1)
- moved B17 46.8 mm to (59.7, -21.0)
- moved B16 46.4 mm to (60.8, -19.7)
- moved C5 46.3 mm to (51.9, -8.76)
- moved B15 46.3 mm to (59.9, -18.5)
- moved B3 46.2 mm to (51.1, -25.9)
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Routing:
- net +5V: track 0.00 -> 428.5 mm
- net GND: track 0.00 -> 154.2 mm, vias 0 -> 62
- net /D5~~_DAT: track 0.00 -> 35.8 mm
- net /LED/D5~~_DAT_OUT: track 0.00 -> 31.6 mm
- net /RESET: track 0.00 -> 31.3 mm
- net /MOSI: track 0.00 -> 25.6 mm
- net /SCK: track 0.00 -> 21.6 mm
- net /MISO: track 0.00 -> 13.6 mm
- net /Vin: track 0.00 -> 12.8 mm
- net /12V: track 0.00 -> 11.6 mm
- net /PB6: track 0.00 -> 10.4 mm
- net /PB7: track 0.00 -> 8.30 mm
- net Net-(D15-Pad2): track 0.00 -> 8.00 mm
- net Net-(D7-Pad2): track 0.00 -> 7.98 mm
- net Net-(D6-Pad2): track 0.00 -> 7.98 mm
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- added copper zone on B.Cu, net GND
Other:
- net class 10 mils added: clearance 0.2, trace_width 0.254, via_dia 0.8, via_drill 0.4
- net class 15 mils added: clearance 0.2, trace_width 0.381, via_dia 0.8, via_drill 0.4
- net class 20 mils added: clearance 0.2, trace_width 0.508, via_dia 0.8, via_drill 0.4
- net class 25 mils added: clearance 0.2, trace_width 0.635, via_dia 0.8, via_drill 0.4

Commit message: added qwiic I2C conn for ToF sensor
Parts:
- added C11: C_NPOL, halo:C_0805_2012Metric, F.Cu at (-95.9, 8.38)
- added C12: C_NPOL, halo:C_0805_2012Metric, F.Cu at (-57.8, 8.38)
- added C13: C_NPOL, halo:C_0805_2012Metric, F.Cu at (-19.7, 8.38)
- added C14: C_NPOL, halo:C_0805_2012Metric, F.Cu at (18.4, 8.38)
- added C15: C_NPOL, halo:C_0805_2012Metric, F.Cu at (56.5, 8.38)
- added C16: C_NPOL, halo:C_0805_2012Metric, F.Cu at (94.6, 8.38)
- added P5: qwiic, halo:PinSocket_1x04_P2.54mm_Vertical_SMD_Pin1Left, F.Cu at (0.00, 28.8)
- moved C10 11.3 mm to (76.1, -18.3), turned to 90 degrees
- moved D31 9.22 mm to (5.59, -18.0)
- moved J1 7.22 mm to (11.3, -25.3)
- moved P1 5.01 mm to (-83.3, -12.7)
- moved C4 2.55 mm to (38.5, -11.7)
- moved C3 2.54 mm to (41.0, -11.7)
- moved P4 2.54 mm to (87.6, -12.7)
- moved R8 2.41 mm to (63.0, -27.1)
- moved D34 2.16 mm to (60.6, -27.1)
- moved X1 1.99 mm to (58.0, -9.65)
- moved C5 1.93 mm to (53.7, -9.53)
- moved C6 1.82 mm to (62.4, -9.53)
- moved C1 1.65 mm to (44.7, -10.8)
- moved B12 1.65 mm to (48.9, -12.3)
- moved P3 1.34 mm to (68.5, -18.2), turned to 0 degrees
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Routing:
- net +5V: track 428.5 -> 647.6 mm
- net /D5~~_DAT: track 35.8 -> 207.3 mm
- net /D6~~_CLK: track 3.73 -> 168.5 mm
- net /SDA: track 5.42 -> 89.5 mm, vias 0 -> 2
- net /SCL: track 5.35 -> 85.6 mm, vias 0 -> 2
- net /D4_MODE: track 5.52 -> 83.9 mm, vias 0 -> 2
- net /TXD: track 1.87 -> 45.7 mm
- net /RESET: track 31.3 -> 68.2 mm, vias 0 -> 3
- net /Vusb: track 3.61 -> 39.4 mm
- net /RXD: track 1.85 -> 36.6 mm
- net /CC1: track 0.00 -> 31.9 mm
- net /CC2: track 0.00 -> 21.8 mm
- net /SBU2: track 0.00 -> 20.5 mm
- net /D+: track 0.00 -> 20.0 mm, vias 0 -> 2
- net /SBU1: track 0.00 -> 19.4 mm
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
Commit message: added PCB review needed
Parts:
- added G***: LOGO, halo:logo_halo, F.Cu at (-51.4, 19.1)
- added G***: LOGO, halo:logo_wyolum, F.Cu at (51.4, 22.2)
- C1, C7: footprint Capacitor_SMD:CP_Elec_4x5.8 -> halo:CP_Elec_4x5.8
- C10, C2, C3, C4, C5, C6, C8, C9: footprint Capacitor_SMD:C_0805_2012Metric -> halo:C_0805_2012Metric
- D1, D10, D11, D12, D13, D14, D15, D16, D17, D18, D19, D2, D20, D21, D22, D23, D24, D25, D26, D27, D28, D29, D3, D30, D4, D5, D6, D7, D8, D9: footprint LED_SMD:LED_WS2812B_PLCC4_5.0x5.0mm_P3.2mm -> halo:LED_WS2812B_PLCC4_5.0x5.0mm_P3.2mm
- D31, D32: footprint Diode_SMD:D_SMB-SMC_Universal_Handsoldering -> halo:D_SMB-SMC_Universal_Handsoldering
- D33, D34: footprint LED_SMD:LED_0805_2012Metric -> halo:LED_0805_2012Metric
- J1: footprint Connector_PinSocket_2.54mm:PinSocket_1x08_P2.54mm_Vertical_SMD_Pin1Left -> halo:PinSocket_1x08_P2.54mm_Vertical_SMD_Pin1Left
- J2: footprint Connector_USB:USB_C_Receptacle_Amphenol_12401610E4-2A_CircularHoles -> halo:AMPHENOL_12401610E4#2A
- J3: footprint Connector_BarrelJack:BarrelJack_CUI_PJ-036AH-SMT_Horizontal -> halo:BarrelJack_CUI_PJ-036AH-SMT_Horizontal
- P1, P4: footprint Connector_PinSocket_2.54mm:PinSocket_1x04_P2.54mm_Vertical_SMD_Pin1Left -> halo:PinSocket_1x04_P2.54mm_Vertical_SMD_Pin1Left
- P2: footprint Connector_PinHeader_2.54mm:PinHeader_1x06_P2.54mm_Vertical_SMD_Pin1Left -> halo:PinHeader_1x06_P2.54mm_Vertical_SMD_Pin1Left
- P3: footprint Connector_PinHeader_2.54mm:PinHeader_2x03_P2.54mm_Vertical_SMD -> halo:PinHeader_2x03_P2.54mm_Vertical_SMD
- R1, R2, R3, R4, R5, R6, R7, R8: footprint Resistor_SMD:R_0805_2012Metric -> halo:R_0805_2012Metric
- SC1, SC2, SC3, SC4, SC5, SC6, SC7, SC8: footprint MountingHole:MountingHole_3.2mm_M3_Pad_Via -> halo:MountingHole_3.2mm_M3_Pad_Via
- SW1: footprint Button_Switch_SMD:SW_Push_1P1T_NO_6x6mm_H9.5mm -> halo:SW_Push_1P1T_NO_6x6mm_H9.5mm
- SW2: footprint Connector_PinHeader_2.54mm:PinHeader_1x02_P2.54mm_Vertical_SMD_Pin1Left -> halo:PinHeader_1x02_P2.54mm_Vertical_SMD_Pin1Left
- U1: footprint Package_QFP:TQFP-32_7x7mm_P0.8mm -> halo:TQFP-32_7x7mm_P0.8mm
- U2: footprint Package_TO_SOT_SMD:SOT-223-3_TabPin2 -> halo:SOT-223-3_TabPin2
- moved R1 13.4 mm to (43.2, -23.9), turned to 180 degrees
- moved C9 8.47 mm to (26.2, -27.1), turned to 270 degrees
- moved P2 7.73 mm to (32.5, -34.4), turned to 270 degrees
- moved J2 4.45 mm to (10.2, -32.4)
- moved SW1 3.89 mm to (32.4, -22.9), turned to 180 degrees
- moved B12 1.02 mm to (48.9, -13.3)
- moved C11 0.99 mm to (-96.9, 8.38), turned to 90 degrees
- moved C13 0.99 mm to (-20.7, 8.38), turned to 90 degrees
- moved C14 0.99 mm to (17.4, 8.38), turned to 90 degrees
- moved C16 0.99 mm to (93.6, 8.38), turned to 90 degrees
- moved C12 0.94 mm to (-58.7, 8.38), turned to 90 degrees
- moved C15 0.91 mm to (55.6, 8.38), turned to 90 degrees
- turned D31 to 180 degrees
- turned D32 to 0 degrees
- turned D33 to 270 degrees
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Connections:
- R7 pad 2: Net-(D33-Pad1) -> Net-(D33-PadA)
- R8 pad 2: Net-(D34-Pad1) -> Net-(D34-PadA)
Routing:
- net +5V: track 647.6 -> 703.5 mm
- net /RESET: track 68.2 -> 54.4 mm
- net /RXD: track 36.6 -> 48.1 mm
- net /D4_MODE: track 83.9 -> 93.0 mm
- net /SDA: track 89.5 -> 95.6 mm
- net Net-(D33-PadA): track 0.00 -> 5.69 mm
- net GND: track 153.0 -> 158.6 mm, vias 68 -> 69
- net Net-(D33-Pad1): track 5.31 -> 0.00 mm
- net /D5~~_DAT: track 207.3 -> 202.9 mm
- net Net-(D34-PadA): track 0.00 -> 2.42 mm
- net Net-(D34-Pad1): track 2.42 -> 0.00 mm
- net /D3~~: track 3.06 -> 1.97 mm
- net /CC1: track 31.9 -> 32.9 mm
- net /CC2: track 21.8 -> 22.8 mm
- net /D6~~_CLK: track 168.5 -> 167.6 mm
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- added copper zone on F.Cu, net +5V
Other:
- net class Default: trace_width 0.25 -> 0.254

Commit message: Gerber BoM ready
Parts:
- removed G***: LOGO, halo:logo_halo
- removed G***: LOGO, halo:logo_wyolum
- added D35: LED_PWR, halo:LED_0805_2012Metric, F.Cu at (107.2, 81.5)
- added D36: LED_BLNK, halo:LED_0805_2012Metric, F.Cu at (200.3, 74.5)
- added G1: logo_halo, halo:logo_halo, B.Cu at (76.2, 101.6)
- added G2: logo_kicad, halo:logo_KiCad_12mm_SilkScreen, F.Cu at (76.2, 120.7)
- added G3: logo_OSH, halo:logo_OSHW_11.4x12mm_SilkScreen, F.Cu at (203.2, 120.7)
- added G4: logo_wyolum, halo:logo_wyolum, B.Cu at (203.2, 101.6)
- C11, C12, C13, C14, C15, C16: value C_NPOL -> 100nF
- C5, C6: value 22p -> 20pF
- D31, D32: value DIODESCH -> WS2812B; footprint halo:D_SMB-SMC_Universal_Handsoldering -> halo:LED_WS2812B_PLCC4_5.0x5.0mm_P3.2mm
- D33: value LED_PWR -> DIODESCH; footprint halo:LED_0805_2012Metric -> halo:D_SMB
- D34: value LED_BLNK -> DIODESCH; footprint halo:LED_0805_2012Metric -> halo:D_SMB
- J1: footprint halo:PinSocket_1x08_P2.54mm_Vertical_SMD_Pin1Left -> halo:PinHeader_2x04_P2.54mm_Vertical_SMD
- J2: footprint halo:AMPHENOL_12401610E4#2A -> halo:USB_C_XKB_U262-241N-4BV64_v2
- J3: footprint halo:BarrelJack_CUI_PJ-036AH-SMT_Horizontal -> halo:barrel_jack_DC-005-5A-2_5-SMT
- P5: footprint halo:PinSocket_1x04_P2.54mm_Vertical_SMD_Pin1Left -> halo:sparkfun_apds_9960_smd
- SW2: footprint halo:PinHeader_1x02_P2.54mm_Vertical_SMD_Pin1Left -> halo:PinHeader_2x02_P2.54mm_Vertical_SMD
- X1: footprint halo:Xtal_SMD4 -> halo:Crystal_SMD_3225-4Pin_3.2x2.5mm
- moved D32 290.8 mm to (257.8, 101.6), turned to 90 degrees
- moved D31 272.3 mm to (250.2, 101.6), turned to 90 degrees
- moved D33 205.6 mm to (145.3, 83.6), turned to 180 degrees
- moved SW2 183.2 mm to (152.4, 137.2)
- moved C5 174.2 mm to (194.8, 92.7), turned to 270 degrees
- moved C4 173.1 mm to (178.1, 90.7)
- moved C3 173.1 mm to (180.6, 90.7)
- moved C12 173.0 mm to (81.3, 110.0)
- moved C10 172.8 mm to (215.9, 83.3)
- moved C15 172.8 mm to (195.3, 110.0)
- moved U1 172.7 mm to (193.0, 83.3)
- moved X1 172.7 mm to (198.1, 91.4)
- moved B8 172.7 mm to (191.8, 77.0)
- moved P4 172.7 mm to (227.3, 88.9)
- moved R4 172.7 mm to (189.5, 91.9)
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Connections:
- D30 pad 2: /LED/D5~~_DAT_OUT -> Net-(D30-Pad2)
- D33 pad A: Net-(D33-PadA) -> /Vusb
- D33 pad K: GND -> +5V
- D34 pad A: Net-(D34-PadA) -> /Vin
- D34 pad K: GND -> /12V
- J3 pad 3: (no net) -> GND
- R7 pad 2: Net-(D33-PadA) -> Net-(D35-PadA)
- R8 pad 2: Net-(D34-PadA) -> Net-(D36-PadA)
- X1 pad 3: GND -> /PB7
Routing:
- net /Vusb: track 40.0 -> 62.5 mm, vias 0 -> 3
- net GND: track 158.6 -> 180.7 mm, vias 69 -> 79
- net +5V: track 703.5 -> 725.6 mm
- net /SCL: track 84.8 -> 98.2 mm
- net /CC2: track 22.8 -> 36.2 mm, vias 0 -> 2
- net /Vin: track 12.8 -> 25.2 mm
- net /D5~~_DAT: track 202.9 -> 214.7 mm, vias 0 -> 2
- net /D4_MODE: track 93.0 -> 83.0 mm
- net /D-: track 12.6 -> 20.8 mm
- net Net-(D31-Pad2): track 0.00 -> 8.00 mm
- net Net-(D30-Pad2): track 0.00 -> 7.97 mm
- net /LED/D5~~_DAT_OUT: track 33.0 -> 40.4 mm
- net /SBU2: track 19.7 -> 26.1 mm
- net Net-(D33-PadA): track 5.69 -> 0.00 mm
- net Net-(D35-PadA): track 0.00 -> 5.58 mm
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Other:
- outline, holes or cut-outs redrawn
- net class 7 mils added: clearance 0.127, trace_width 0.1778, via_dia 0.8, via_drill 0.4
- rule trace_min: 0.2 -> 0.1524

Commit message: Gerber BoM Position files for JLCpcb
Parts:
- removed J1: USB_header, halo:PinHeader_2x04_P2.54mm_Vertical_SMD
- added B21: I_O, halo:breakout_smd, F.Cu at (231.8, 90.2)
- added C17: 100nF, halo:C_0805_2012Metric, F.Cu at (142.7, 67.1)
- added C18: 100nF, halo:C_0805_2012Metric, F.Cu at (143.8, 117.9)
- added C19: 100nF, halo:C_0805_2012Metric, F.Cu at (109.5, 85.6)
- added C20: 100nF, halo:C_0805_2012Metric, F.Cu at (177.2, 72.4)
- added P6: USB_header, halo:PinHeader_2x04_P2.54mm_Vertical_SMD, F.Cu at (151.9, 72.6)
- added R10: 0E, halo:R_0805_2012Metric, F.Cu at (206.4, 92.7)
- added R9: 0E, halo:R_0805_2012Metric, F.Cu at (203.8, 92.7)
- C1, C7: value 10uF -> 22uF
- C10, C2, C9: value 100n -> 100nF
- D33, D34: value DIODESCH -> MBRS240LT3G
- J2: value USB_C_Receptacle_USB2.0 -> USB4110-GF-A; footprint halo:USB_C_XKB_U262-241N-4BV64_v2 -> halo:GCT_USB4110-GF-A
- P1: value LED -> LED_IN
- moved B20 139.9 mm to (60.7, 90.2)
- moved R7 5.95 mm to (104.9, 81.5)
- moved R5 2.01 mm to (145.0, 67.1), turned to 90 degrees
- moved R6 1.91 mm to (158.8, 67.1)
- moved J2 0.28 mm to (151.9, 60.7)
Connections:
- net /LED/D5~~_DAT_OUT renamed /LED/DAT_OUT
- B20 pad 1: /D6~~_CLK -> /CLK
- D1 pad 4: /D5~~_DAT -> /DAT
- P1 pad 2: /D5~~_DAT -> /DAT
- P1 pad 3: /D6~~_CLK -> /CLK
- P5 pad 1: GND -> Net-(P5-Pad1)
- P5 pad 2: +5V -> GND
- P5 pad 3: /SDA -> +5V
- P5 pad 4: /SCL -> /SDA
Routing:
- net GND: track 180.7 -> 789.8 mm, vias 79 -> 92
- net /DAT: track 0.00 -> 203.3 mm, vias 0 -> 2
- net /D5~~_DAT: track 214.7 -> 12.6 mm, vias 2 -> 0
- net /CLK: track 0.00 -> 156.9 mm
- net /D6~~_CLK: track 168.0 -> 13.9 mm
- net /SBU2: track 26.1 -> 9.19 mm
- net /CC2: track 36.2 -> 21.9 mm, vias 2 -> 0
- net /CC1: track 37.4 -> 23.5 mm
- net /RXD: track 48.3 -> 37.9 mm
- net /TXD: track 46.2 -> 38.4 mm
- net /LED/DAT_OUT: track 40.4 -> 48.1 mm
- net /SBU1: track 15.9 -> 9.82 mm
- net Net-(B21-Pad1): track 0.00 -> 6.10 mm
- net /RESET: track 54.7 -> 60.7 mm, vias 3 -> 4
- net +5V: track 725.6 -> 730.5 mm
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