File: kicad/halo.sch (KiCad schematic (older format))
At the start: 60 parts, among them J1 USB_header, J2 USB_C_Receptacle_USB2.0, J3 12V_DC, P1 LED, P2 FTDI, P3 SPI, SW1 RST, SW2 MODE, U1 ATMEGA328, U2 LM1117-5.0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

Commit message: added qwiic I2C conn for ToF sensor
Parts:
- added P5: qwiic, halo:PinSocket_1x04_P2.54mm_Vertical_SMD_Pin1Left, symbol halo:CONN_4
Connections:
- wire segments 194 -> 202
Other:
- moved on the sheet: P1
Changed lines of the file:
@@
 U 1 1 4DCB971F
 P 3875 7050
-F 0 "P2" H 3875 6825 60  0000 C CNN
-F 1 "FTDI" H 3875 6700 60  0000 C CNN
+F 0 "P2" H 3825 6700 60  0000 C CNN
+F 1 "FTDI" V 3875 7050 50  0000 C CNB
 F 2 "Connector_PinHeader_2.54mm:PinHeader_1x06_P2.54mm_Vertical_SMD_Pin1Left" H 3875 7050 60  0001 C CNN
 F 3 "" H 3875 7050 60  0001 C CNN
@@
 	8850 2750 9950 2750
 Wire Wire Line
-	9950 2750 9950 2125
+	9950 2750 9950 2525
 Text Label 8950 800  0    50   ~ 0
 5V
@@
 U 1 1 5FA38811
 P 1125 7200
-F 0 "P3" H 1175 7522 50  0000 C CNN
-F 1 "SPI" H 1175 7431 50  0000 C CNN
+F 0 "P3" H 1125 7400 50  0000 C CNN
+F 1 "SPI" V 1175 7200 50  0000 C CNB
 F 2 "Connector_PinHeader_2.54mm:PinHeader_2x03_P2.54mm_Vertical_SMD" H 1125 7200 50  0001 C CNN
 F 3 "~" H 1125 7200 50  0001 C CNN
@@
 U 1 1 5FAFBE8C
 P 2050 7325
-F 0 "C10" H 1950 7200 50  0000 L CNN
+F 0 "C10" H 1900 7200 50  0000 L CNN
 F 1 "100n" H 1850 7450 50  0000 L CNN
 F 2 "Capacitor_SMD:C_0805_2012Metric" H 2050 7350 60  0001 C CNN
@@
 Connection ~ 9750 2125
 Wire Wire Line
-	9750 2125 9750 2650
+	9750 2125 9750 2425
 $Comp
 L halo:CONN_4 P1
 U 1 1 5FB9549F
-P 10825 3700
-F 0 "P1" H 10959 3745 50  0000 L CNN
-F 1 "LED" H 10959 3654 50  0000 L CNN
-F 2 "Connector_PinSocket_2.54mm:PinSocket_1x04_P2.54mm_Vertical_SMD_Pin1Left" H 10825 3700 60  0001 C CNN
-F 3 "" H 10825 3700 60  0000 C CNN
-	1    10825 3700
-	1    0    0    -1
-$EndComp
-Wire Wire Line
-	8850 3650 10475 3650
-Wire Wire Line
-	8850 3750 10475 3750
-Wire Wire Line
-	10475 3850 10375 3850
+P 10925 3700
+F 0 "P1" H 10825 3950 50  0000 L CNN
+F 1 "LED" V 10925 3625 50  0000 L CNB
+F 2 "Connector_PinSocket_2.54mm:PinSocket_1x04_P2.54mm_Vertical_SMD_Pin1Left" H 10925 3700 60  0001 C CNN
+F 3 "" H 10925 3700 60  0000 C CNN
+	1    10925 3700
+	1    0    0    -1
+$EndComp
+Wire Wire Line
+	8850 3650 10575 3650
+Wire Wire Line
+	8850 3750 10575 3750
+Wire Wire Line
+	10575 3850 10375 3850
 Wire Wire Line
 	10375 3850 10375 4975
@@
 Connection ~ 10150 4975
 Wire Wire Line
-	10475 3550 10375 3550
-Wire Wire Line
-	10375 3550 10375 800
+	10575 3550 10375 3550
+Wire Wire Line
+	10375 3550 10375 2325
 Wire Wire Line
 	10375 800  10150 800
@@
 Wire Wire Line
 	2125 1400 3325 1400
+$Comp
+L halo:CONN_4 P5
+U 1 1 5FA65C4B
+P 10925 2375
+F 0 "P5" H 10825 2625 50  0000 L CNN
+F 1 "qwiic" V 10925 2375 50  0000 C CNB
+F 2 "halo:PinSocket_1x04_P2.54mm_Vertical_SMD_Pin1Left" H 10925 2375 60  0001 C CNN
+F 3 "" H 10925 2375 60  0000 C CNN
+	1    10925 2375
+	1    0    0    -1
+$EndComp
+Wire Wire Line
+	10575 2325 10375 2325
+Connection ~ 10375 2325
+Wire Wire Line
+	10375 2325 10375 800
+Wire Wire Line
+	10575 2425 9750 2425
+Connection ~ 9750 2425
+Wire Wire Line
+	9750 2425 9750 2650
+Wire Wire Line
+	10575 2525 9950 2525
+Connection ~ 9950 2525
+Wire Wire Line
+	9950 2525 9950 2125
+Wire Wire Line
+	10575 2225 10475 2225
+Wire Wire Line
+	10475 2225 10475 2700
+$Comp
+L power:GND #PWR05
+U 1 1 5FA99C4C
+P 10475 2700
+F 0 "#PWR05" H 10475 2700 30  0001 C CNN
+F 1 "GND" H 10475 2630 30  0001 C CNN
+F 2 "" H 10475 2700 60  0001 C CNN
+F 3 "" H 10475 2700 60  0001 C CNN
+	1    10475 2700
+	1    0    0    -1
+$EndComp
+Text Label 10475 2225 0    50   ~ 0
+GND
 $EndSCHEMATC

Commit message: added PCB review needed
Parts:
- C1, C7: footprint Capacitor_SMD:CP_Elec_4x5.8 -> halo:CP_Elec_4x5.8
- C10, C2, C3, C4, C5, C6, C8, C9: footprint Capacitor_SMD:C_0805_2012Metric -> halo:C_0805_2012Metric
- D31, D32: footprint Diode_SMD:D_SMB-SMC_Universal_Handsoldering -> halo:D_SMB-SMC_Universal_Handsoldering
- D33, D34: footprint LED_SMD:LED_0805_2012Metric -> halo:LED_0805_2012Metric
- J1: footprint Connector_PinSocket_2.54mm:PinSocket_1x08_P2.54mm_Vertical_SMD_Pin1Left -> halo:PinSocket_1x08_P2.54mm_Vertical_SMD_Pin1Left
- J2: footprint Connector_USB:USB_C_Receptacle_Amphenol_12401610E4-2A_CircularHoles -> halo:AMPHENOL_12401610E4#2A; symbol Connector:USB_C_Receptacle_USB2.0 -> halo:USB_C_Receptacle_USB2.0
- J3: footprint Connector_BarrelJack:BarrelJack_CUI_PJ-036AH-SMT_Horizontal -> halo:BarrelJack_CUI_PJ-036AH-SMT_Horizontal
- P1: footprint Connector_PinSocket_2.54mm:PinSocket_1x04_P2.54mm_Vertical_SMD_Pin1Left -> halo:PinSocket_1x04_P2.54mm_Vertical_SMD_Pin1Left
- P2: footprint Connector_PinHeader_2.54mm:PinHeader_1x06_P2.54mm_Vertical_SMD_Pin1Left -> halo:PinHeader_1x06_P2.54mm_Vertical_SMD_Pin1Left
- P3: footprint Connector_PinHeader_2.54mm:PinHeader_2x03_P2.54mm_Vertical_SMD -> halo:PinHeader_2x03_P2.54mm_Vertical_SMD
- R1, R2, R3, R4, R5, R6, R7, R8: footprint Resistor_SMD:R_0805_2012Metric -> halo:R_0805_2012Metric
- SC1, SC2, SC3, SC4, SC5, SC6, SC7, SC8: footprint MountingHole:MountingHole_3.2mm_M3_Pad_Via -> halo:MountingHole_3.2mm_M3_Pad_Via
- SW1: footprint Button_Switch_SMD:SW_Push_1P1T_NO_6x6mm_H9.5mm -> halo:SW_Push_1P1T_NO_6x6mm_H9.5mm
- SW2: footprint Connector_PinHeader_2.54mm:PinHeader_1x02_P2.54mm_Vertical_SMD_Pin1Left -> halo:PinHeader_1x02_P2.54mm_Vertical_SMD_Pin1Left
- U1: footprint Package_QFP:TQFP-32_7x7mm_P0.8mm -> halo:TQFP-32_7x7mm_P0.8mm
- U2: footprint Package_TO_SOT_SMD:SOT-223-3_TabPin2 -> halo:SOT-223-3_TabPin2

Commit message: Gerber BoM ready
Parts:
- removed J3: 12V_DC, halo:BarrelJack_CUI_PJ-036AH-SMT_Horizontal, symbol halo:Jack-DC
- removed SW2: MODE, halo:PinHeader_1x02_P2.54mm_Vertical_SMD_Pin1Left, symbol halo:SW_PUSH
- added G1: logo_halo, halo:logo_halo, symbol halo:logo_halo
- added G2: logo_kicad, halo:logo_KiCad_12mm_SilkScreen, symbol halo:logo_kicad
- added G3: logo_OSH, halo:logo_OSHW_11.4x12mm_SilkScreen, symbol halo:logo_OSH
- added G4: logo_wyolum, halo:logo_wyolum, symbol halo:logo_wyolum
- added J3: 12V_DC, halo:barrel_jack_DC-005-5A-2_5-SMT, symbol Connector:Barrel_Jack_Switch
- added SW2: MODE, halo:PinHeader_2x02_P2.54mm_Vertical_SMD, symbol halo:SW_Push_Dual
- C5, C6: value 22p -> 20pF
- D33: renamed from D31; footprint halo:D_SMB-SMC_Universal_Handsoldering -> halo:D_SMB
- D34: renamed from D32; footprint halo:D_SMB-SMC_Universal_Handsoldering -> halo:D_SMB
- J1: footprint halo:PinSocket_1x08_P2.54mm_Vertical_SMD_Pin1Left -> halo:PinHeader_2x04_P2.54mm_Vertical_SMD
- J2: footprint halo:AMPHENOL_12401610E4#2A -> halo:USB_C_XKB_U262-241N-4BV64_v2
- P5: footprint halo:PinSocket_1x04_P2.54mm_Vertical_SMD_Pin1Left -> halo:sparkfun_apds_9960_smd
- X1: footprint halo:Xtal_SMD4 -> halo:Crystal_SMD_3225-4Pin_3.2x2.5mm
- renumbered D33 to D35, D34 to D36
Connections:
- net D4_MODE: now also SW2.2, SW2.4
- net GND: now also J3.2, J3.3, SW2.1, SW2.3
- net Vin: now also J3.1
Other:
- note added: "Mating Plug\nOD = 5.5 mm\nID = 2.5 mm"

Commit message: Gerber BoM Position files for JLCpcb
Parts:
- removed J2: USB_C_Receptacle_USB2.0, halo:USB_C_XKB_U262-241N-4BV64_v2, symbol halo:USB_C_Receptacle_USB2.0
- removed P5: qwiic, halo:sparkfun_apds_9960_smd, symbol halo:CONN_4
- added C17, C18, C19, C20: 100nF, halo:C_0805_2012Metric, symbol halo:C_NPOL
- added J2: USB4110-GF-A, halo:GCT_USB4110-GF-A, symbol halo:USB4110-GF-A
- added P5: qwiic, halo:sparkfun_apds_9960_smd, symbol halo:CONN_01x06
- added R10, R9: 0E, halo:R_0805_2012Metric, symbol halo:R2
- C1, C7: value 10uF -> 22uF
- C10, C2, C9: value 100n -> 100nF
- D33, D34: value DIODESCH -> MBRS240LT3G
- P1: value LED -> LED_IN; symbol halo:CONN_4 -> halo:CONN_01x04
- P2: symbol halo:CONN_6 -> halo:CONN_01x06
- P3: symbol halo:Conn_02x03_Odd_Even -> halo:CONN_02x03_Odd_Even
- P6: renamed from J1; symbol halo:Conn_01x08 -> halo:CONN_02x04_Odd_Even
Connections:
- net +5V: now also C18.1, C19.1, C20.1, P5.3 (Pin_3)
- net CC1: now also P6.5 (Pin_5), J2.A5 (CC1); no longer P6.2 (Pin_2)
- net CC2: now also J2.B5 (CC2)
- net D+: now also P6.6 (Pin_6), J2.A6 (DP1), J2.B6 (DP2); no longer P6.5 (Pin_5)
- net D-: now also J2.A7 (DN1), J2.B7 (DN2)
- net D5~~_DAT: now also R9.2; no longer P1.2 (P2)
- net D6~~_CLK: now also R10.2; no longer P1.3 (P3)
- net GND: now also P6.7 (Pin_7), C17.2, C18.2, C19.2, C20.2, J2.A1/B12 (GND), J2.B1/A12 (GND__1), J2.S1 (GND__2), J2.S2 (GND__3), J2.S3 (GND__4), J2.S4 (GND__5), P5.2 (Pin_2); no longer P6.8 (Pin_8)
- net SBU1: now also P6.2 (Pin_2), J2.A8 (SBU1); no longer P6.6 (Pin_6)
- net SBU2: now also P6.8 (Pin_8), J2.B8 (SBU2); no longer P6.7 (Pin_7)
- net SCL: now also P5.5 (Pin_5)
- net SDA: now also P5.4 (Pin_4)
- net Vusb: now also C17.1, J2.A4/B9 (VBUS), J2.B4/A9 (VBUS__1)
- new net CLK: P1.3 (Pin_3), R10.1
- new net DAT: P1.2 (Pin_2), R9.1
- no-connect marks 0 -> 2
Other:
- note added: "SPI / PROG Header"
- note removed: "ISP/PROG Header"
- moved on the sheet: B1, B2, C7, C8, D34, D35, D36, J3, P1, P2, P6, R2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
