File: kicad_v2/halo.sch (KiCad schematic (older format))
At the start: 73 parts, among them J2 USB4110-GF-A, J3 12V_DC, P1 LED_IN1, P2 FTDI, P3 SPI, P5 qwiic, P6 USB_header, SW1 RST, SW2 MODE, U1 ATMEGA328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

Commit message: halo_v2 almost done
Parts:
- added B21: I_O, halo:breakout_smd, symbol halo:I_O
- added G5: logo_halo, halo:logo_halo_10mm, symbol halo:logo_halo
- added J1: 12V_DC, halo:conn_barrel, symbol Connector:Barrel_Jack_Switch
- added P7: generic, halo:generic_apds_9960_smd, symbol halo:Conn_01x05
- C1, C27, C7: footprint halo:CP_Elec_10x10 -> halo:CP_Elec_6.3x7.7
- P1: value LED_IN1 -> LED_IN
Connections:
- net +5V: now also P7.1 (Pin_1)
- net GND: now also J1.2, J1.3, P7.2 (Pin_2)
- net SCL: now also P7.3 (Pin_3)
- net SDA: now also P7.4 (Pin_4)
- net Vin: now also J1.1
- new net: B21.1, P7.5 (Pin_5)
Other:
- note added: "Locking Barrel\nSocket"
- note added: "Mating Plug\nOD = 5.5 mm\nID = 2.1 mm"
- note removed: "Mating Plug\nOD = 5.5 mm\nID = 2.5 mm"
- moved on the sheet: B1, B10, B11, B12, B13, B14, B15, B16, B17, B18, B19, B2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
