File: kicad_v2/halo.kicad_pcb (KiCad board)
At the start: 2 copper layers, 243.8 x 66.2 mm, 151 parts, among them J2 USB4110-GF-A, J3 12V_DC, P1 LED_IN1, P2 FTDI, P3 SPI, P4 LED_OUT, P5 qwiic, P6 USB_header, SW1 RST, SW2 MODE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

Commit message: halo_v2 almost done
Parts:
- added B21: I_O, halo:breakout_smd, F.Cu at (152.3, 113.0)
- added G5: logo_halo, halo:logo_halo_10mm, F.Cu at (216.3, 119.9)
- added J1: 12V_DC, halo:conn_barrel, F.Cu at (139.7, 68.6)
- added P7: generic, halo:generic_apds_9960_smd, F.Cu at (148.6, 118.1)
- C1, C27, C7: footprint halo:CP_Elec_10x10 -> halo:CP_Elec_6.3x7.7
- G4: moved to F.Cu
- P1: value LED_IN1 -> LED_IN
- moved G4 134.9 mm to (69.2, 117.5), turned to 0 degrees
- moved D65 125.9 mm to (250.2, 98.4)
- moved D66 116.2 mm to (250.2, 104.8)
- moved D30 114.3 mm to (128.3, 104.8), turned to 0 degrees
- moved D28 106.9 mm to (120.7, 98.4)
- moved D29 106.9 mm to (128.3, 98.4), turned to 0 degrees
- moved D41 106.7 mm to (158.8, 98.4), turned to 0 degrees
- moved G2 104.2 mm to (188.6, 104.1)
- moved C12 99.5 mm to (62.2, 114.3), turned to 90 degrees
- moved D42 99.3 mm to (158.8, 104.8), turned to 0 degrees
- moved D43 99.3 mm to (166.4, 104.8)
- moved SC1 98.3 mm to (41.4, 63.5)
- moved D57 96.5 mm to (219.7, 98.4)
- moved D64 96.5 mm to (242.6, 98.4), turned to 180 degrees
- moved D45 91.4 mm to (174.0, 98.4), turned to 0 degrees
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Routing:
- net +5V: track 53.2 -> 1013.9 mm, vias 2 -> 7
- net GND: track 114.6 -> 477.7 mm, vias 19 -> 130
- net /D5~~_DAT: track 0.00 -> 136.5 mm, vias 0 -> 2
- net /D6~~_CLK: track 0.00 -> 134.0 mm, vias 0 -> 2
- net /SCL: track 0.00 -> 113.6 mm, vias 0 -> 2
- net /SDA: track 0.00 -> 112.7 mm, vias 0 -> 2
- net /RESET: track 0.00 -> 80.3 mm, vias 0 -> 4
- net /DAT: track 0.00 -> 70.2 mm, vias 0 -> 2
- net /LED_2/DAT_OUT2: track 3.30 -> 53.1 mm, vias 0 -> 2
- net /D4_MODE: track 0.00 -> 42.3 mm, vias 0 -> 2
- net /TXD: track 3.30 -> 41.1 mm, vias 0 -> 2
- net /RXD: track 3.30 -> 36.7 mm, vias 0 -> 2
- net /MOSI: track 0.00 -> 29.2 mm
- net /MISO: track 0.00 -> 26.7 mm
- net /SCK: track 0.00 -> 25.2 mm, vias 0 -> 2
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- added copper zone on F.Cu, net +5V
Other:
- board size 243.8 x 66.2 mm -> 243.8 x 66.3 mm
- net class 30 mils added: clearance 0.2, trace_width 0.762, via_dia 0.8, via_drill 0.4
- net class 50 mils added: clearance 0.2, trace_width 1.27, via_dia 0.8, via_drill 0.4
- board text added: "ver 2"

Commit message: halo_v2 JLCpcb files ready
Parts:
- moved U1 0.13 mm to (190.5, 78.7)
Routing:
- net /Vusb: track 40.0 -> 78.8 mm, vias 2 -> 4
